File: Project/IO_device.kicad_pcb (KiCad board)
At the start: 4 copper layers, 160 x 100 mm, 274 parts, among them J1 Screw_Terminal_01x02, J10 Screw_Terminal_01x02, J11 Screw_Terminal_01x02, J12 Screw_Terminal_01x02, J13 USB_C_Receptacle_PowerOnly_6P, J14 Conn_01x01, J15 Screw_Terminal_01x03, J17 Conn_01x01, J18 Conn_01x01, J19 Conn_01x01, J2 Screw_Terminal_01x02, J3 Screw_Terminal_01x02, J4 Screw_Terminal_01x02, J5 Screw_Terminal_01x02, J6 Screw_Terminal_01x02, J7 Screw_Terminal_01x02, J8 Screw_Terminal_01x02, J9 Screw_Terminal_01x02, K1 SDT-S-103DMR,000, K2 SDT-S-103DMR,000, K3 SDT-S-103DMR,000, K4 SDT-S-103DMR,000, Q1 BC847, Q11 BC847, Q12 BC847, Q13 AO3400A, Q2 BC847, Q3 BC847, Q4 BC847, Q5 2SCR587D3, Q6 2SCR587D3, Q7 AO3400A, Q8 AO3400A, Q9 AO3400A, U1 MCP4728, U10 74HC240D, U11 TL071, U12 TL071, U13 IL300-DEFG-X007T, U14 IL300-DEFG-X007T, U15 TL071, U16 TL071, U17 MCP3208T-BI/SL, U18 CNY173SR2VM, U19 CNY173SR2VM, U2 TL071, U20 CNY173SR2VM, U21 CNY173SR2VM, U22 MM74HC14M, U24 TBA1-0522E, U25 TBA1-0522E, U26 TBA1-0522E, U27 ADM2483xRW, U28 NUCLEO-L152RE, U3 TL071, U4 IL300-DEFG-X007T, U5 IL300-DEFG-X007T, U6 TL071, U7 TL071, U8 TL071, U9 TL071

Commit message: Add files via upload
Parts:
- moved C56 11.6 mm to (111.6, 146.8)
- moved C81 2.34 mm to (130.5, 137.0), turned to 180 degrees
- moved C51 2.13 mm to (119.8, 131.0)
- moved C22 0.60 mm to (177.1, 105.5)
- turned C5 to 180 degrees
Routing:
- net E5V: track 88.8 -> 146.2 mm
- net GNDD: track 469.7 -> 524.9 mm, vias 30 -> 241
- net Net-(Q13-G): track 34.8 -> 56.0 mm
- net -12VA: track 247.6 -> 257.3 mm
- net +3.3V: track 515.3 -> 524.2 mm
- net -12V: track 114.2 -> 121.5 mm
- net +12V: track 254.2 -> 250.5 mm
- net ADC_CH0: track 57.9 -> 55.0 mm
- net GND3: track 278.9 -> 280.3 mm
- added copper zone on B.Cu, net GNDD
- added copper zone on F.Cu, net GNDD
Other:
- board text added: "Eevertti Pylkkä"
